Commit message: working urdf

File: onine_urdf/urdf/onine.urdf (robot description, URDF)
Before this commit: robot visual, 10 links, 9 joints
Links:
- added link base_footprint
- added link camera_link; visual box size=0.06 0.28 0.06
- added link wheel1; visual cylinder length=0.05 radius=.05
- added link wheel2; visual cylinder length=0.05 radius=.05
- added link wheel3; visual cylinder length=0.05 radius=.05
- added link wheel4; visual cylinder length=0.05 radius=.05
- link base_link: geometry visual box size=0.33 0.23 0.15
- link torso_link: geometry visual box size=0.134 0.125 0.005
- link vertical_link: geometry visual box size=0.02 0.02 1.21
Joints:
- added joint base_link_joint: type fixed, parent base_footprint, child base_link, origin xyz=0 0 0.171 rpy=0 0 0, axis 0 0 1
- added joint camera_link_joint: type fixed, parent vertical_link, child camera_link, origin xyz=0 0 1.21 rpy=0 0.5585 0, axis 0 0 1
- added joint wheel1_joint: type fixed, parent base_footprint, child wheel1, origin xyz=0.11 0.17 0.05 rpy=0 0 0, axis 0 0 1
- added joint wheel2_joint: type fixed, parent base_footprint, child wheel2, origin xyz=0.11 -0.17 0.05 rpy=0 0 0, axis 0 0 1
- added joint wheel3_joint: type fixed, parent base_footprint, child wheel3, origin xyz=-0.11 0.17 0.05 rpy=0 0 0, axis 0 0 1
- added joint wheel4_joint: type fixed, parent base_footprint, child wheel4, origin xyz=-0.11 -0.17 0.05 rpy=0 0 0, axis 0 0 1
- joint base_joint: origin xyz=0 0 0 rpy=0 0 0 -> xyz=0.015 0 0 rpy=0 0 0
- joint torso_joint: limit lower=0.18 upper=1.04 effort=1000.0 velocity=1.0 -> lower=0.185 upper=0.6 effort=1000.0 velocity=0.108; origin xyz=0.095 0 0 rpy=0 0 0 -> xyz=0.078 0 0 rpy=0 0 0; parent base_link -> vertical_link
- joint vertical_joint: origin xyz=0 0 0.54 rpy=0 0 0 -> xyz=-0.013 0 0 rpy=0 0 0

Commit message: changed from belt to threaded rod design

File: onine_urdf/urdf/onine.urdf (robot description, URDF)
Before this commit: robot onine, 16 links, 15 joints
Links:
- added link rod_link; visual cylinder length=.985 radius=.004
- link camera_link: geometry visual box size=0.06 0.28 0.035
- link torso_link: geometry visual box size=0.15 0.145 0.005
- link vertical_link: geometry visual box size=0.02 0.02 1.025
Joints:
- added joint rod_joint: type fixed, parent vertical_link, child rod_link, origin xyz=0.045 0 0 rpy=0 0 0, axis 0 0 1
- joint base_joint: origin xyz=0.015 0 0 rpy=0 0 0 -> xyz=0.0075 0 0 rpy=0 0 0
- joint camera_link_joint: origin xyz=0 0 1.21 rpy=0 0.5585 0 -> xyz=0 0 1.08 rpy=0 0.593412 0
- joint torso_joint: limit lower=0.185 upper=0.6 effort=1000.0 velocity=0.108 -> lower=0.21 upper=0.9 effort=1000.0 velocity=0.108; origin xyz=0.078 0 0 rpy=0 0 0 -> xyz=0.08 0 0 rpy=0 0 0; parent vertical_link -> rod_link
- joint vertical_joint: origin xyz=-0.013 0 0 rpy=0 0 0 -> xyz=-0.035 0 0 rpy=0 0 0

Commit message: adjusted rod_joint transform to fix rviz color problem

File: onine_urdf/urdf/onine.urdf (robot description, URDF)
Before this commit: robot visual, 17 links, 16 joints
Joints:
- joint rod_joint: origin xyz=0.045 0 0 rpy=0 0 0 -> xyz=0.045 0 0.0000000001 rpy=0 0 0

Commit message: partially rearrange links for collada compatibility

File: onine_urdf/urdf/onine.urdf (robot description, URDF)
Before this commit: robot onine, 17 links, 16 joints
Links:
- link rod_link: geometry visual cylinder length=0.825 radius=.004
Joints:
- joint camera_link_joint: origin xyz=0 0 1.08 rpy=0 0.593412 0 -> xyz=-0.001 0 0.5675 rpy=0 0.593412 0
- joint rod_joint: origin xyz=0.045 0 0.0000000001 rpy=0 0 0 -> xyz=0.045 0 0 rpy=0 0 0
- joint torso_joint: origin xyz=0.08 0 0 rpy=0 0 0 -> xyz=0.08 0 -0.5125 rpy=0 0 0
- joint vertical_joint: origin xyz=-0.035 0 0 rpy=0 0 0 -> xyz=-0.035 0 0.5125 rpy=0 0 0

Commit message: fixed stl package path

File: onine_urdf/urdf/onine.urdf (robot description, URDF)
Before this commit: robot onine, 17 links, 16 joints
Links:
- link braccio_base_link: geometry visual mesh filename=package://onine_urdf/stl/braccio_base.stl scale=0.001 0.001 0.001
- link elbow_link: geometry visual mesh filename=package://onine_urdf/stl/braccio_elbow.stl scale=0.001 0.001 0.001
- link left_gripper_link: geometry visual mesh filename=package://onine_urdf/stl/braccio_left_gripper.stl scale=0.001 0.001 0.001
- link right_gripper_link: geometry visual mesh filename=package://onine_urdf/stl/braccio_right_gripper.stl scale=0.001 0.001 0.001
- link shoulder_link: geometry visual mesh filename=package://onine_urdf/stl/braccio_shoulder.stl scale=0.001 0.001 0.001
- link wrist_pitch_link: geometry visual mesh filename=package://onine_urdf/stl/braccio_wrist_pitch.stl scale=0.001 0.001 0.001
- link wrist_roll_link: geometry visual mesh filename=package://onine_urdf/stl/braccio_wrist_roll.stl scale=0.001 0.001 0.001

Commit message: sync all angle limits with physical robot

File: onine_urdf/urdf/onine.urdf (robot description, URDF)
Before this commit: robot onine, 17 links, 16 joints
Joints:
- joint base_joint: limit lower=0.0 upper=3.1416 effort=1000.0 velocity=1.0 -> lower=0.0872665 upper=3.1416 effort=1000.0 velocity=1.0
- joint wrist_pitch_joint: limit lower=0 upper=3.1416 effort=1000.0 velocity=1.0 -> lower=0.0872665 upper=3.1416 effort=1000.0 velocity=1.0

Commit message: added horizontal beam that's holding on the threaded rod

File: onine_urdf/urdf/onine.urdf (robot description, URDF)
Before this commit: robot onine, 17 links, 16 joints
Links:
- added link beam_link; visual box size=0.02 0.07 0.025
Joints:
- added joint beam_link_joint: type fixed, parent vertical_link, child beam_link, origin xyz=0.021 0 0.3975 rpy=0 0 0, axis 0 0 1

Commit message: corrected camera transform

File: onine_urdf/urdf/onine.urdf (robot description, URDF)
Before this commit: robot onine, 18 links, 17 joints
Joints:
- joint camera_link_joint: origin xyz=-0.001 0 0.5675 rpy=0 0.593412 0 -> xyz=-0.001 0.03 0.5675 rpy=0 0.593412 0

Commit message: redo urdf

File: onine_urdf/urdf/onine.urdf (robot description, URDF)
Before this commit: robot onine, 18 links, 17 joints
Links:
- link left_gripper_link: geometry visual box size=0.006 0.002 0.075
- link right_gripper_link: geometry visual box size=0.006 0.002 0.075
Joints:
- joint base_joint: axis 0 0 -1 -> 0 0 1; limit lower=0.0872665 upper=3.1416 effort=1000.0 velocity=1.0 -> lower=-1.570796 upper=1.570796 effort=1000.0 velocity=1.0; origin xyz=0.0075 0 0 rpy=0 0 0 -> xyz=0 0 0.0756 rpy=0 0 0
- joint elbow_joint: axis 1 0 0 -> 0 1 0; limit lower=0 upper=3.1416 effort=1000.0 velocity=1.0 -> lower=-1.570796 upper=1.570796 effort=1000.0 velocity=1.0; origin xyz=0 0 0.125 rpy=-1.5708 0 0 -> xyz=0 0 0.13 rpy=0 0 0
- joint gripper_joint: axis 0 -1 0 -> 0 1 0; child right_gripper_link -> left_gripper_link; limit lower=1.217 upper=1.5708 effort=1000.0 velocity=1.0 -> lower=0.002 upper=0.04 effort=1000.0 velocity=1.0; origin xyz=0.010 0 0.03 rpy=0 0 0 -> xyz=-0.0035 0 0.078 rpy=0 0 0; type revolute -> prismatic
- joint shoulder_joint: axis 1 0 0 -> 0 1 0; limit lower=0.2618 upper=2.8798 effort=1000.0 velocity=1.0 -> lower=-1.308997 upper=1.308997 effort=1000.0 velocity=1.0; origin xyz=0 -.002 0.072 rpy=-1.5708 0 0 -> xyz=0 0 0 rpy=0 0 0
- joint sub_gripper_joint: axis 0 1 0 -> 0 -1 0; child left_gripper_link -> right_gripper_link; limit lower=1.5708 upper=2.7876 effort=1000.0 velocity=1.0 -> lower=-0.002 upper=-0.04 effort=1000.0 velocity=1.0; origin xyz=-0.010 0 0.03 rpy=0 3.1416 0 -> xyz=-0.0035 0 0.078 rpy=0 0 0; type revolute -> prismatic
- joint torso_joint: limit lower=0.21 upper=0.9 effort=1000.0 velocity=0.108 -> lower=0.21 upper=0.9 effort=1000.0 velocity=0.0303875
- joint wrist_pitch_joint: axis 1 0 0 -> 0 1 0; limit lower=0.0872665 upper=3.1416 effort=1000.0 velocity=1.0 -> lower=-1.570796 upper=1.570796 effort=1000.0 velocity=1.0; origin xyz=0 0 0.125 rpy=-1.5708 0 0 -> xyz=0 0 0.125 rpy=0 0 0
- joint wrist_roll_joint: axis 0 0 -1 -> 0 0 1; limit lower=0.0 upper=3.1416 effort=1000.0 velocity=1.0 -> lower=0.000 upper=3.141592 effort=1000.0 velocity=1.0; origin xyz=0 0.0 0.06 rpy=0 0 0 -> xyz=0 0 0.06 rpy=0 0 0

Commit message: working package to match changes in urdf

File: onine_urdf/urdf/onine.urdf (robot description, URDF)
Before this commit: robot onine, 18 links, 17 joints
Joints:
- joint base_joint: limit lower=-1.570796 upper=1.570796 effort=1000.0 velocity=1.0 -> lower=-1.570796 upper=1.4835295 effort=1000.0 velocity=1.0
- joint elbow_joint: origin xyz=0 0 0.13 rpy=0 0 0 -> xyz=0 0 0.125 rpy=0 0 0
- joint sub_gripper_joint: limit lower=-0.002 upper=-0.04 effort=1000.0 velocity=1.0 -> lower=0.002 upper=0.04 effort=1000.0 velocity=1.0

Commit message: changed wrist_roll_link transform

File: onine_urdf/urdf/onine.urdf (robot description, URDF)
Before this commit: robot onine, 18 links, 17 joints
Links:
- link left_gripper_link: geometry visual box size=0.075 0.002 0.006
- link right_gripper_link: geometry visual box size=0.075 0.002 0.006
Joints:
- joint gripper_joint: origin xyz=-0.0035 0 0.078 rpy=0 0 0 -> xyz=.0776 0 0.005 rpy=0 0 0
- joint sub_gripper_joint: origin xyz=-0.0035 0 0.078 rpy=0 0 0 -> xyz=0.0776 0 0.005 rpy=0 0 0
- joint wrist_roll_joint: axis 0 0 1 -> 1 0 0; origin xyz=0 0 0.06 rpy=0 0 0 -> xyz=0 0 0.06 rpy=0 -1.570796 0

Commit message: added tool_link

File: onine_urdf/urdf/onine.urdf (robot description, URDF)
Before this commit: robot onine, 18 links, 17 joints
Links:
- added link tool_link
Joints:
- added joint tool_link_joint: type fixed, parent wrist_roll_link, child tool_link, origin xyz=0.08 0 0 rpy=0 0 0, axis 1 0 0

Commit message: calibrated kinect

File: onine_urdf/urdf/onine.urdf (robot description, URDF)
Before this commit: robot onine, 19 links, 18 joints
Joints:
- joint camera_link_joint: origin xyz=-0.001 0.03 0.5675 rpy=0 0.593412 0 -> xyz=-0.001 0.065 0.5675 rpy=0 0.593412 0

Commit message: changed joint limits after fixing arm

File: onine_urdf/urdf/onine.urdf (robot description, URDF)
Before this commit: robot onine, 19 links, 18 joints
Joints:
- joint base_joint: limit lower=-1.570796 upper=1.4835295 effort=1000.0 velocity=1.0 -> lower=-1.396263 upper=1.570796 effort=1000.0 velocity=1.0

Commit message: changed base joint limits to match arm

File: onine_urdf/urdf/onine.urdf (robot description, URDF)
Before this commit: robot onine, 19 links, 18 joints
Joints:
- joint base_joint: limit lower=-1.396263 upper=1.570796 effort=1000.0 velocity=1.0 -> lower=-1.309 upper=1.570796 effort=1000.0 velocity=1.0
- joint camera_link_joint: origin xyz=-0.001 0.065 0.5675 rpy=0 0.593412 0 -> xyz=0.00 0.055 0.5675 rpy=0 0.593412 0
- joint wrist_roll_joint: axis 1 0 0 -> -1 0 0
