Commit message: renamed onine_urdf to onine_description to follow standards

File: onine_description/urdf/onine.urdf (robot description, URDF)
Before this commit: robot onine, 19 links, 18 joints
Links:
- link braccio_base_link: geometry visual mesh filename=package://onine_description/stl/braccio_base.stl scale=0.001 0.001 0.001
- link elbow_link: geometry visual mesh filename=package://onine_description/stl/braccio_elbow.stl scale=0.001 0.001 0.001
- link shoulder_link: geometry visual mesh filename=package://onine_description/stl/braccio_shoulder.stl scale=0.001 0.001 0.001
- link wrist_pitch_link: geometry visual mesh filename=package://onine_description/stl/braccio_wrist_pitch.stl scale=0.001 0.001 0.001
- link wrist_roll_link: geometry visual mesh filename=package://onine_description/stl/braccio_wrist_roll.stl scale=0.001 0.001 0.001

Commit message: sync hardware changes

File: onine_description/urdf/onine.urdf (robot description, URDF)
Before this commit: robot onine, 19 links, 18 joints
Joints:
- joint base_joint: limit lower=-1.309 upper=1.570796 effort=1000.0 velocity=1.0 -> lower=-1.13446 upper=1.65806 effort=1000.0 velocity=1.0
- joint camera_link_joint: origin xyz=0.00 0.055 0.5675 rpy=0 0.593412 0 -> xyz=0.00 0.03 0.5675 rpy=0 0.593412 0
- joint elbow_joint: limit lower=-1.570796 upper=1.570796 effort=1000.0 velocity=1.0 -> lower=-1.22173 upper=1.65806 effort=1000.0 velocity=1.0
- joint shoulder_joint: limit lower=-1.308997 upper=1.308997 effort=1000.0 velocity=1.0 -> lower=-1.309 upper=1.309 effort=1000.0 velocity=1.0
- joint wrist_pitch_joint: limit lower=-1.570796 upper=1.570796 effort=1000.0 velocity=1.0 -> lower=-1.6507 upper=1.53589 effort=1000.0 velocity=1.0

Commit message: revert to prev camera transform

File: onine_description/urdf/onine.urdf (robot description, URDF)
Before this commit: robot onine, 19 links, 18 joints
Joints:
- joint camera_link_joint: origin xyz=0.00 0.03 0.5675 rpy=0 0.593412 0 -> xyz=0.00 0.055 0.5675 rpy=0 0.593412 0
